File: CircuitDesign/SmartwaterTank/receiver.sch (EAGLE design)
At the start: 13 parts

Commit message: sync mqtt receive with transmitter data
Connections:
- net N$5: now also NODE1.D1; no longer NODE1.TX
Changed lines of the file:
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@@
 <pinref part="SG1" gate="G$1" pin="1"/>
 <wire x1="99.06" y1="167.64" x2="63.5" y2="167.64" width="0.1524" layer="91"/>
-<wire x1="63.5" y1="167.64" x2="63.5" y2="149.86" width="0.1524" layer="91"/>
-<pinref part="NODE1" gate="G$1" pin="TX"/>
-<wire x1="63.5" y1="149.86" x2="60.96" y2="149.86" width="0.1524" layer="91"/>
-<junction x="63.5" y="149.86"/>
-<junction x="63.5" y="167.64"/>
+<wire x1="63.5" y1="167.64" x2="63.5" y2="177.8" width="0.1524" layer="91"/>
+<pinref part="NODE1" gate="G$1" pin="D1"/>
+<wire x1="63.5" y1="177.8" x2="60.96" y2="177.8" width="0.1524" layer="91"/>
 </segment>
 </net>
